File: PSUtap_eval_LT6105/PSUtap_eval_LT6105.sch (KiCad schematic (older format))
At the start: 9 parts, among them J1 Conn_01x03_Male, U1 LT6105-Amplifier_Current

Commit message: updated project with custom library
Parts:
- U1: symbol lt6105-amplifier:LT6105-Amplifier_Current -> PSUtap_eval_LT6105-rescue:LT6105-Amplifier_Current-lt6105-amplifier
Changed lines of the file:
@@
 $EndComp
 $Comp
-L lt6105-amplifier:LT6105-Amplifier_Current U1
+L PSUtap_eval_LT6105-rescue:LT6105-Amplifier_Current-lt6105-amplifier U1
 U 1 1 606E1D6E
 P 5500 3200
