File: PSUtap_digital/PSUtap_digital.sch (KiCad schematic (older format))
At the start: 80 parts, among them J1 USB_B_Micro, J2 ADC_board_SPI, J3 SD_card_SPI, J4 Screen_SPI, SW1 Up, SW2 Down, SW3 Left, SW4 Right, SW5 B, SW6 A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

Commit message: Updated analog board PCB and started digital board PSB
Parts:
- C1, C12, C24, C26, C3, C5, C9: footprint Capacitor_SMD:C_0805_2012Metric_Pad1.15x1.40mm_HandSolder -> Capacitor_SMD:C_0603_1608Metric_Pad1.05x0.95mm_HandSolder
Changed lines of the file:
@@
 F 0 "C1" H 2088 1446 50  0000 L CNN
 F 1 "22u" H 2088 1355 50  0000 L CNN
-F 2 "Capacitor_SMD:C_0805_2012Metric_Pad1.15x1.40mm_HandSolder" H 2000 1400 50  0001 C CNN
+F 2 "Capacitor_SMD:C_0603_1608Metric_Pad1.05x0.95mm_HandSolder" H 2000 1400 50  0001 C CNN
 F 3 "~" H 2000 1400 50  0001 C CNN
 	1    2000 1400
@@
 F 0 "C3" H 4042 2046 50  0000 L CNN
 F 1 "2.2u" H 4042 1955 50  0000 L CNN
-F 2 "Capacitor_SMD:C_0805_2012Metric_Pad1.15x1.40mm_HandSolder" H 3950 2000 50  0001 C CNN
+F 2 "Capacitor_SMD:C_0603_1608Metric_Pad1.05x0.95mm_HandSolder" H 3950 2000 50  0001 C CNN
 F 3 "~" H 3950 2000 50  0001 C CNN
 	1    3950 2000
@@
 F 0 "C5" H 5538 2396 50  0000 L CNN
 F 1 "22u" H 5538 2305 50  0000 L CNN
-F 2 "Capacitor_SMD:C_0805_2012Metric_Pad1.15x1.40mm_HandSolder" H 5450 2350 50  0001 C CNN
+F 2 "Capacitor_SMD:C_0603_1608Metric_Pad1.05x0.95mm_HandSolder" H 5450 2350 50  0001 C CNN
 F 3 "~" H 5450 2350 50  0001 C CNN
 	1    5450 2350
@@
 F 0 "C26" H 3292 7246 50  0000 L CNN
 F 1 "1u" H 3292 7155 50  0000 L CNN
-F 2 "Capacitor_SMD:C_0805_2012Metric_Pad1.15x1.40mm_HandSolder" H 3200 7200 50  0001 C CNN
+F 2 "Capacitor_SMD:C_0603_1608Metric_Pad1.05x0.95mm_HandSolder" H 3200 7200 50  0001 C CNN
 F 3 "~" H 3200 7200 50  0001 C CNN
 	1    3200 7200
@@
 F 0 "C24" H 4988 7196 50  0000 L CNN
 F 1 "22u" H 4988 7105 50  0000 L CNN
-F 2 "Capacitor_SMD:C_0805_2012Metric_Pad1.15x1.40mm_HandSolder" H 4900 7150 50  0001 C CNN
+F 2 "Capacitor_SMD:C_0603_1608Metric_Pad1.05x0.95mm_HandSolder" H 4900 7150 50  0001 C CNN
 F 3 "~" H 4900 7150 50  0001 C CNN
 	1    4900 7150
@@
 F 0 "C9" H 2242 3296 50  0000 L CNN
 F 1 "1u" H 2242 3205 50  0000 L CNN
-F 2 "Capacitor_SMD:C_0805_2012Metric_Pad1.15x1.40mm_HandSolder" H 2150 3250 50  0001 C CNN
+F 2 "Capacitor_SMD:C_0603_1608Metric_Pad1.05x0.95mm_HandSolder" H 2150 3250 50  0001 C CNN
 F 3 "~" H 2150 3250 50  0001 C CNN
 	1    2150 3250
@@
 F 0 "C12" H 5138 3296 50  0000 L CNN
 F 1 "4.7u" H 5138 3205 50  0000 L CNN
-F 2 "Capacitor_SMD:C_0805_2012Metric_Pad1.15x1.40mm_HandSolder" H 5050 3250 50  0001 C CNN
+F 2 "Capacitor_SMD:C_0603_1608Metric_Pad1.05x0.95mm_HandSolder" H 5050 3250 50  0001 C CNN
 F 3 "~" H 5050 3250 50  0001 C CNN
 	1    5050 3250

Commit message: Caching of project footprints
KiCad "digital rescue" of externally sourced footprints into cache
Parts:
- U1: symbol Battery_Management:LT1512 -> PSUtap_digital-rescue:LT1512-Battery_Management
- U3: symbol Battery_Management:Si6926ADQ -> PSUtap_digital-rescue:Si6926ADQ-Battery_Management
Changed lines of the file:
@@
 $EndComp
 $Comp
-L Battery_Management:LT1512 U1
+L PSUtap_digital-rescue:LT1512-Battery_Management U1
 U 1 1 5F3DB73C
 P 2850 2200
@@
 $EndComp
 $Comp
-L Battery_Management:Si6926ADQ U3
+L PSUtap_digital-rescue:Si6926ADQ-Battery_Management U3
 U 1 1 5F5A4436
 P 8200 2200

Commit message: Removed PCB copies, added xtal to ADC in analog board, finished digital board's PCB
Parts:
- C1, C5: footprint Capacitor_SMD:C_0603_1608Metric_Pad1.05x0.95mm_HandSolder -> Capacitor_SMD:C_0805_2012Metric_Pad1.15x1.40mm_HandSolder
- C12: Notes (none) -> CM03X5R475M06AH055
- U1: symbol PSUtap_digital-rescue:LT1512-Battery_Management -> Battery_Management:LT1512
- U3: symbol PSUtap_digital-rescue:Si6926ADQ-Battery_Management -> Battery_Management:Si6926ADQ
Other:
- moved on the sheet: C13
Changed lines of the file:
@@
 $EndComp
 $Comp
-L PSUtap_digital-rescue:LT1512-Battery_Management U1
+L Battery_Management:LT1512 U1
 U 1 1 5F3DB73C
 P 2850 2200
@@
 F 0 "C1" H 2088 1446 50  0000 L CNN
 F 1 "22u" H 2088 1355 50  0000 L CNN
-F 2 "Capacitor_SMD:C_0603_1608Metric_Pad1.05x0.95mm_HandSolder" H 2000 1400 50  0001 C CNN
-F 3 "~" H 2000 1400 50  0001 C CNN
+F 2 "Capacitor_SMD:C_0805_2012Metric_Pad1.15x1.40mm_HandSolder" H 2000 1400 50  0001 C CNN
+F 3 "GRM219R61C226ME15L" H 2000 1400 50  0001 C CNN
 	1    2000 1400
 	1    0    0    -1
@@
 F 0 "C5" H 5538 2396 50  0000 L CNN
 F 1 "22u" H 5538 2305 50  0000 L CNN
-F 2 "Capacitor_SMD:C_0603_1608Metric_Pad1.05x0.95mm_HandSolder" H 5450 2350 50  0001 C CNN
-F 3 "~" H 5450 2350 50  0001 C CNN
+F 2 "Capacitor_SMD:C_0805_2012Metric_Pad1.15x1.40mm_HandSolder" H 5450 2350 50  0001 C CNN
+F 3 "GRM219R61C226ME15L" H 5450 2350 50  0001 C CNN
 	1    5450 2350
 	1    0    0    -1
@@
 $EndComp
 $Comp
-L PSUtap_digital-rescue:Si6926ADQ-Battery_Management U3
+L Battery_Management:Si6926ADQ U3
 U 1 1 5F5A4436
 P 8200 2200
@@
 !RDY
 $Comp
-L MCU_Microchip_ATmega:ATmega328P-AU U5
-U 1 1 5F73246F
-P 4850 4850
-F 0 "U5" H 4400 3400 50  0000 C CNN
-F 1 "ATmega328P-AU" H 4450 3300 50  0000 C CNN
-F 2 "Package_QFP:TQFP-32_7x7mm_P0.8mm" H 4850 4850 50  0001 C CIN
-F 3 "http://ww1.microchip.com/downloads/en/DeviceDoc/ATmega328_P%20AVR%20MCU%20with%20picoPower%20Technology%20Data%20Sheet%2040001984A.pdf" H 4850 4850 50  0001 C CNN
-	1    4850 4850
-	1    0    0    -1
-$EndComp
-$Comp
 L power:GND #PWR030
 U 1 1 5F8FBB37
@@
 	4850 6400 4850 6350
 Wire Wire Line
-	4850 3350 4850 3150
-Wire Wire Line
 	4850 3150 4950 3150
-Wire Wire Line
-	4950 3350 4950 3150
 Connection ~ 4950 3150
 Wire Wire Line
@@
 F 2 "Capacitor_SMD:C_0603_1608Metric_Pad1.05x0.95mm_HandSolder" H 5050 3250 50  0001 C CNN
 F 3 "~" H 5050 3250 50  0001 C CNN
+F 4 "CM03X5R475M06AH055" H 5050 3250 50  0001 C CNN "Notes"
 	1    5050 3250
 	1    0    0    -1
@@
 L Device:C_Small C13
 U 1 1 5F978F34
-P 5350 3250
-F 0 "C13" H 5442 3296 50  0000 L CNN
-F 1 "100n" H 5442 3205 50  0000 L CNN
-F 2 "Capacitor_SMD:C_0603_1608Metric_Pad1.05x0.95mm_HandSolder" H 5350 3250 50  0001 C CNN
-F 3 "~" H 5350 3250 50  0001 C CNN
-	1    5350 3250
-	1    0    0    -1
-$EndComp
-$Comp
-L power:GND #PWR016
-U 1 1 5F9792A7
-P 5550 3350
-F 0 "#PWR016" H 5550 3100 50  0001 C CNN
-F 1 "GND" H 5555 3177 50  0000 C CNN
-F 2 "" H 5550 3350 50  0001 C CNN
-F 3 "" H 5550 3350 50  0001 C CNN
-	1    5550 3350
-	1    0    0    -1
-$EndComp
-Wire Wire Line
-	5550 3150 5350 3150
-Wire Wire Line
-	5050 3150 5350 3150
-Connection ~ 5350 3150
-Wire Wire Line
-	5050 3350 5350 3350
-Wire Wire Line
-	5350 3350 5550 3350
-Connection ~ 5350 3350
+P 1800 3250
+F 0 "C13" H 1892 3296 50  0000 L CNN
+F 1 "100n" H 1892 3205 50  0000 L CNN
+F 2 "Capacitor_SMD:C_0603_1608Metric_Pad1.05x0.95mm_HandSolder" H 1800 3250 50  0001 C CNN
+F 3 "~" H 1800 3250 50  0001 C CNN
+	1    1800 3250
+	1    0    0    -1
+$EndComp
 Wire Wire Line
 	5450 5350 5600 5350
@@
 Text Label 2350 5200 0    50   ~ 0
 5Vsup
+Wire Wire Line
+	5050 3150 5550 3150
+Wire Wire Line
+	4950 3350 4950 3150
+Wire Wire Line
+	4850 3350 4850 3150
+$Comp
+L power:GND #PWR016
+U 1 1 5F9792A7
+P 5450 3350
+F 0 "#PWR016" H 5450 3100 50  0001 C CNN
+F 1 "GND" H 5455 3177 50  0000 C CNN
+F 2 "" H 5450 3350 50  0001 C CNN
+F 3 "" H 5450 3350 50  0001 C CNN
+	1    5450 3350
+	1    0    0    -1
+$EndComp
+$Comp
+L MCU_Microchip_ATmega:ATmega328P-AU U5
+U 1 1 5F73246F
+P 4850 4850
+F 0 "U5" H 4400 3400 50  0000 C CNN
+F 1 "ATmega328P-AU" H 4450 3300 50  0000 C CNN
+F 2 "Package_QFP:TQFP-32_7x7mm_P0.8mm" H 4850 4850 50  0001 C CIN
+F 3 "http://ww1.microchip.com/downloads/en/DeviceDoc/ATmega328_P%20AVR%20MCU%20with%20picoPower%20Technology%20Data%20Sheet%2040001984A.pdf" H 4850 4850 50  0001 C CNN
+	1    4850 4850
+	1    0    0    -1
+$EndComp
+Wire Wire Line
+	5450 3350 5050 3350
+Wire Wire Line
+	1800 3350 2150 3350
+Connection ~ 2150 3350
 $EndSCHEMATC

Commit message: updated kicad projects caches
Parts:
- J1: symbol Connector:USB_B_Micro -> PSUtap_digital-rescue:USB_B_Micro-Connector
- U1: symbol Battery_Management:LT1512 -> PSUtap_digital-rescue:LT1512-Battery_Management
- U3: symbol Battery_Management:Si6926ADQ -> PSUtap_digital-rescue:Si6926ADQ-Battery_Management
Changed lines of the file:
@@
 $EndDescr
 $Comp
-L Connector:USB_B_Micro J1
+L PSUtap_digital-rescue:USB_B_Micro-Connector J1
 U 1 1 5F3D1BFD
 P 900 1450
@@
 $EndComp
 $Comp
-L Battery_Management:LT1512 U1
+L PSUtap_digital-rescue:LT1512-Battery_Management U1
 U 1 1 5F3DB73C
 P 2850 2200
@@
 $EndComp
 $Comp
-L Battery_Management:Si6926ADQ U3
+L PSUtap_digital-rescue:Si6926ADQ-Battery_Management U3
 U 1 1 5F5A4436
 P 8200 2200
