File: PSUtap_eval_AD7708/PSUtap_eval_AD7708.sch (KiCad schematic (older format))
At the start: 28 parts, among them J1 Analog_Inputs, J2 Conn_01x02, J3 Conn_01x10_Female, SW1 SW_Push, U1 AD7708-Analog_ADC-PSUtap_anal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, U2 AD780ANZ, Y1 Device_Crystal_Small

Commit message: single-sided evaluation board for AD7708
Parts:
- U1: symbol PSUtap_analog-rescue:AD7708-Analog_ADC-PSUtap_analog-rescue -> PSUtap_eval_AD7708-rescue:AD7708-Analog_ADC-PSUtap_analog-rescue-PSUtap_analog-rescue
- U2: value AD780ANZ -> AD780ARZ
- Y1: symbol PSUtap_analog-cache:Device_Crystal_Small -> PSUtap_eval_AD7708-rescue:Device_Crystal_Small-PSUtap_analog-cache
Changed lines of the file:
@@
 	6000 4450 6000 4400
 $Comp
-L PSUtap_analog-cache:Device_Crystal_Small Y1
+L PSUtap_eval_AD7708-rescue:Device_Crystal_Small-PSUtap_analog-cache Y1
 U 1 1 607338CA
 P 6250 3900
@@
 	1450 1900 1450 1750
 $Comp
-L PSUtap_analog-rescue:AD7708-Analog_ADC-PSUtap_analog-rescue U1
+L PSUtap_eval_AD7708-rescue:AD7708-Analog_ADC-PSUtap_analog-rescue-PSUtap_analog-rescue U1
 U 1 1 6073881A
 P 4900 2550
@@
 P 7700 4850
 F 0 "U2" H 10000 5237 60  0000 C CNN
-F 1 "AD780ANZ" H 10000 5131 60  0000 C CNN
+F 1 "AD780ARZ" H 10000 5131 60  0000 C CNN
 F 2 "Package_SO:SSOP-8_3.9x5.05mm_P1.27mm" H 10000 5090 60  0001 C CNN
 F 3 "" H 7700 4850 60  0000 C CNN
